Commit message: Gravity compensation!

File: lerobot/common/teleoperators/so102_leader/Leader_arm_links.SLDASM/urdf/Leader_arm_links.SLDASM_old_convention.urdf (robot description, URDF)
Before this commit: robot Leader_arm_links.SLDASM, 7 links, 6 joints
Links:
- link base_link: geometry collision mesh filename=package://Leader_arm_links.SLDASM/meshes/base_link.STL; visual mesh filename=package://Leader_arm_links.SLDASM/meshes/base_link.STL
- link link1: geometry collision mesh filename=package://Leader_arm_links.SLDASM/meshes/link1.STL; visual mesh filename=package://Leader_arm_links.SLDASM/meshes/link1.STL
- link link2: geometry collision mesh filename=package://Leader_arm_links.SLDASM/meshes/link2.STL; visual mesh filename=package://Leader_arm_links.SLDASM/meshes/link2.STL
- link link3: geometry collision mesh filename=package://Leader_arm_links.SLDASM/meshes/link3.STL; visual mesh filename=package://Leader_arm_links.SLDASM/meshes/link3.STL
- link link4: geometry collision mesh filename=package://Leader_arm_links.SLDASM/meshes/link4.STL; visual mesh filename=package://Leader_arm_links.SLDASM/meshes/link4.STL
- link link5: geometry collision mesh filename=package://Leader_arm_links.SLDASM/meshes/link5.STL; visual mesh filename=package://Leader_arm_links.SLDASM/meshes/link5.STL
- link link6: geometry collision mesh filename=package://Leader_arm_links.SLDASM/meshes/link6.STL; visual mesh filename=package://Leader_arm_links.SLDASM/meshes/link6.STL
Joints:
- joint joint2: axis 0 0 -1 -> 0 0 1
- joint joint3: axis 0 0 -1 -> 0 0 1
