Commit message: fixed normalize. unnormalize to do

File: lerobot/common/teleoperators/so102_leader/Leader_arm_links.SLDASM/urdf/Leader_arm_links.SLDASM.urdf (robot description, URDF)
Before this commit: robot Leader_arm_links.SLDASM, 7 links, 6 joints
Joints:
- joint joint1: axis 0 0 -1 -> 0 0 1
- joint joint2: axis 0 0 -1 -> 0 0 1
- joint joint3: axis 0 0 -1 -> 0 0 1

Commit message: gravity comp done

File: lerobot/common/teleoperators/so102_leader/Leader_arm_links.SLDASM/urdf/Leader_arm_links.SLDASM.urdf (robot description, URDF)
Before this commit: robot Leader_arm_links.SLDASM, 7 links, 6 joints
Links:
- link link1: mass 0.15375 -> 0.093
Joints:
- joint joint1: axis 0 0 1 -> 0 0 -1
- joint joint2: origin xyz=0 0 0.054 rpy=-1.5795 0 3.1416 -> xyz=0 0 0.054 rpy=-1.5795 3.1416 3.1416
- joint joint4: axis 0 0 -1 -> 0 0 1
- joint joint5: origin xyz=0.0016 -0.0001 0.0592 rpy=3.1416 -1.5708 0 -> xyz=0.0016 -0.0001 0.0592 rpy=0 -1.5708 0
