Commit message: virtually running

File: lerobot/common/teleoperators/kuka_leader/Kuka_leader_description/urdf/Kuka_leader_links.urdf (robot description, URDF)
Before this commit: robot Kuka_leader_links, 7 links, 6 joints
Joints:
- joint Joint1: limit (none) -> lower=-3.14 upper=3.14 effort=100 velocity=1.0; type continuous -> revolute
- joint Joint2: limit (none) -> lower=-3.14 upper=3.14 effort=100 velocity=1.0; type continuous -> revolute
- joint Joint3: limit lower=0 upper=0 effort=0 velocity=0 -> lower=-3.14 upper=3.14 effort=100 velocity=1.0
- joint Joint4: limit (none) -> lower=-3.14 upper=3.14 effort=100 velocity=1.0; type continuous -> revolute
- joint Joint5: limit lower=0 upper=0 effort=0 velocity=0 -> lower=-3.14 upper=3.14 effort=100 velocity=1.0
- joint Joint6: limit (none) -> lower=-3.14 upper=3.14 effort=100 velocity=1.0; type continuous -> revolute
